File: kicad/n720ak/O2.kicad_sch (KiCad schematic)
At the start: 6 parts, among them J1 O2-HEAD-1-PILOT, J2 O2-HEAD-2-COPILOT, J3 O2-HEAD-3-PASS1, J4 O2-HEAD-4-PASS2, J5 O2-REGULATOR, J6 O2-CTRL-HEAD

Commit message: Tie the sheets into one KiCad project with deterministic output
A generated root sheet and project file make the three sheets one
hierarchical KiCad 10 project: 49 connectors, 153 nets. One fewer net than
the sheets separately, because a global label shared between sheets now
joins them - the way an off-sheet flag is meant to mean the same net
everywhere.

UUIDs are now derived deterministically instead of drawn at random. A
generated file under version control that changed every UUID on every
regeneration would show every line modified each time, burying the real
differences. Regenerating an unchanged wire list is now byte-identical.

Reference designators are prefixed per sheet (J101, J201, ...) so they are
unique across the project, and each symbol carries both a standalone and a
hierarchical instance path, so every sheet still verifies on its own and
annotates cleanly inside the project.

Co-Authored-By: Claude Opus 5.5 <noreply@anthropic.com>
Claude-Session: https://claude.ai/code/session_015SpGdnvPFhutgEDurpngu2
Parts:
- removed J1: O2-HEAD-1-PILOT, symbol n720ak:O2-HEAD-1-PILOT
- removed J2: O2-HEAD-2-COPILOT, symbol n720ak:O2-HEAD-2-COPILOT
- removed J3: O2-HEAD-3-PASS1, symbol n720ak:O2-HEAD-3-PASS1
- removed J4: O2-HEAD-4-PASS2, symbol n720ak:O2-HEAD-4-PASS2
- removed J5: O2-REGULATOR, symbol n720ak:O2-REGULATOR
- removed J6: O2-CTRL-HEAD, symbol n720ak:O2-CTRL-HEAD
- added J301: O2-HEAD-1-PILOT, symbol n720ak:O2-HEAD-1-PILOT
- added J302: O2-HEAD-2-COPILOT, symbol n720ak:O2-HEAD-2-COPILOT
- added J303: O2-HEAD-3-PASS1, symbol n720ak:O2-HEAD-3-PASS1
- added J304: O2-HEAD-4-PASS2, symbol n720ak:O2-HEAD-4-PASS2
- added J305: O2-REGULATOR, symbol n720ak:O2-REGULATOR
- added J306: O2-CTRL-HEAD, symbol n720ak:O2-CTRL-HEAD
Connections:
- net CG: now also J301.1, J302.1, J303.1, J304.1, J305.1
- net GMA245 J1-44: now also J306.9
- net Ground: now also J306.14
- net Switch Dimmer: now also J306.21
- net VP-X J10-8: now also J306.1
- new net: J304.2, J305.6, J306.2
- new net: J304.3, J306.4
- new net: J304.4, J306.22
- new net: J304.5, J306.10
- new net: J303.2, J306.3
- new net: J303.3, J306.5
- new net: J303.4, J306.23
- new net: J303.5, J306.11
- new net: J301.2, J306.15
- new net: J301.3, J306.17
- new net: J301.4, J306.25
- new net: J301.5, J306.13
- new net: J302.2, J306.16
- new net: J302.3, J306.18
- new net: J302.4, J306.24
- new net: J302.5, J306.12
- new net: J305.2, J305.9, J306.19
- new net: J305.8, J306.20
- new net: J305.5, J306.6
Changed lines of the file:
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@@
 	(symbol (lib_id "n720ak:O2-HEAD-1-PILOT") (at 220.98 48.26 0) (unit 1)
 		(in_bom yes) (on_board yes) (dnp no)
-		(property "Reference" "J1" (at 220.98 38.1 0) (effects (font (size 1.27 1.27))))
+		(property "Reference" "J301" (at 220.98 38.1 0) (effects (font (size 1.27 1.27))))
 		(property "Value" "O2-HEAD-1-PILOT" (at 220.98 58.42 0) (effects (font (size 1.27 1.27))))
-		(instances (project "n720ak" (path "/4de5817a-edd4-4ce1-8195-4c7a9df7fa0f" (reference "J1") (unit 1)))))
+		(instances (project "n720ak"
+			(path "/68f123fe-0a64-579b-8b4e-10fd39426bfa" (reference "J301") (unit 1))
+			(path "/05ae3897-9dd7-5bc2-b238-7f217081554a/7e6d20c8-2457-5371-8684-7a70b4f29f82" (reference "J301") (unit 1)))))
 	(symbol (lib_id "n720ak:O2-HEAD-2-COPILOT") (at 220.98 71.12 0) (unit 1)
 		(in_bom yes) (on_board yes) (dnp no)
-		(property "Reference" "J2" (at 220.98 60.96 0) (effects (font (size 1.27 1.27))))
+		(property "Reference" "J302" (at 220.98 60.96 0) (effects (font (size 1.27 1.27))))
 		(property "Value" "O2-HEAD-2-COPILOT" (at 220.98 81.28 0) (effects (font (size 1.27 1.27))))
-		(instances (project "n720ak" (path "/4de5817a-edd4-4ce1-8195-4c7a9df7fa0f" (reference "J2") (unit 1)))))
+		(instances (project "n720ak"
+			(path "/68f123fe-0a64-579b-8b4e-10fd39426bfa" (reference "J302") (unit 1))
+			(path "/05ae3897-9dd7-5bc2-b238-7f217081554a/7e6d20c8-2457-5371-8684-7a70b4f29f82" (reference "J302") (unit 1)))))
 	(symbol (lib_id "n720ak:O2-HEAD-3-PASS1") (at 220.98 93.98 0) (unit 1)
 		(in_bom yes) (on_board yes) (dnp no)
-		(property "Reference" "J3" (at 220.98 83.82 0) (effects (font (size 1.27 1.27))))
+		(property "Reference" "J303" (at 220.98 83.82 0) (effects (font (size 1.27 1.27))))
 		(property "Value" "O2-HEAD-3-PASS1" (at 220.98 104.14 0) (effects (font (size 1.27 1.27))))
-		(instances (project "n720ak" (path "/4de5817a-edd4-4ce1-8195-4c7a9df7fa0f" (reference "J3") (unit 1)))))
+		(instances (project "n720ak"
+			(path "/68f123fe-0a64-579b-8b4e-10fd39426bfa" (reference "J303") (unit 1))
+			(path "/05ae3897-9dd7-5bc2-b238-7f217081554a/7e6d20c8-2457-5371-8684-7a70b4f29f82" (reference "J303") (unit 1)))))
 	(symbol (lib_id "n720ak:O2-HEAD-4-PASS2") (at 220.98 116.84 0) (unit 1)
 		(in_bom yes) (on_board yes) (dnp no)
-		(property "Reference" "J4" (at 220.98 106.68 0) (effects (font (size 1.27 1.27))))
+		(property "Reference" "J304" (at 220.98 106.68 0) (effects (font (size 1.27 1.27))))
 		(property "Value" "O2-HEAD-4-PASS2" (at 220.98 127.0 0) (effects (font (size 1.27 1.27))))
-		(instances (project "n720ak" (path "/4de5817a-edd4-4ce1-8195-4c7a9df7fa0f" (reference "J4") (unit 1)))))
+		(instances (project "n720ak"
+			(path "/68f123fe-0a64-579b-8b4e-10fd39426bfa" (reference "J304") (unit 1))
+			(path "/05ae3897-9dd7-5bc2-b238-7f217081554a/7e6d20c8-2457-5371-8684-7a70b4f29f82" (reference "J304") (unit 1)))))
 	(symbol (lib_id "n720ak:O2-REGULATOR") (at 220.98 140.97 0) (unit 1)
 		(in_bom yes) (on_board yes) (dnp no)
-		(property "Reference" "J5" (at 220.98 129.54 0) (effects (font (size 1.27 1.27))))
+		(property "Reference" "J305" (at 220.98 129.54 0) (effects (font (size 1.27 1.27))))
 		(property "Value" "O2-REGULATOR" (at 220.98 152.4 0) (effects (font (size 1.27 1.27))))
-		(instances (project "n720ak" (path "/4de5817a-edd4-4ce1-8195-4c7a9df7fa0f" (reference "J5") (unit 1)))))
+		(instances (project "n720ak"
+			(path "/68f123fe-0a64-579b-8b4e-10fd39426bfa" (reference "J305") (unit 1))
+			(path "/05ae3897-9dd7-5bc2-b238-7f217081554a/7e6d20c8-2457-5371-8684-7a70b4f29f82" (reference "J305") (unit 1)))))
 	(symbol (lib_id "n720ak:O2-CTRL-HEAD") (at 50.8 93.98 0) (unit 1)
 		(in_bom yes) (on_board yes) (dnp no)
-		(property "Reference" "J6" (at 50.8 35.56 0) (effects (font (size 1.27 1.27))))
+		(property "Reference" "J306" (at 50.8 35.56 0) (effects (font (size 1.27 1.27))))
 		(property "Value" "O2-CTRL-HEAD" (at 50.8 152.4 0) (effects (font (size 1.27 1.27))))
-		(instances (project "n720ak" (path "/4de5817a-edd4-4ce1-8195-4c7a9df7fa0f" (reference "J6") (unit 1)))))
+		(instances (project "n720ak"
+			(path "/68f123fe-0a64-579b-8b4e-10fd39426bfa" (reference "J306") (unit 1))
+			(path "/05ae3897-9dd7-5bc2-b238-7f217081554a/7e6d20c8-2457-5371-8684-7a70b4f29f82" (reference "J306") (unit 1)))))
 	(wire (pts (xy 60.96 40.64) (xy 71.12 40.64)) (stroke (width 0) (type default)))
 	(wire (pts (xy 60.96 43.18) (xy 210.82 43.18)) (stroke (width 0) (type default)))
