File: kicad/n720ak/PWR.kicad_sch (KiCad schematic)
At the start: 24 parts, among them J1 VP-X J2, J10 ALTERNATOR, J11 KEYSWITCH, J12 ENGINE START, J13 ANN ECU PWR PRI (GRN), J14 ANN ECU PWR SEC (GRN), J15 ANN FUEL PUMP 1 (GRN), J16 ANN FUEL PUMP 2 (AMB), J17 ANN ECU FAULT PRI (RED), J18 ANN ECU FAULT SEC (RED), J19 PILOT-SW-PANEL DB15, J2 COPILOT-SW-PANEL DB15, J20 START CONTACTOR 1, J21 START CONTACTOR 2, J22 FUEL PUMP CHANGEOVER RELAY, J23 FUEL PUMP MODE, J24 START BAT SEL, J3 VP-X J1, J4 VP-X J12, J5 VP-X J10, J6 ESS BUS, J7 BATT 1, J8 BATT 2, J9 BUS MANAGER

Commit message: Tie the sheets into one KiCad project with deterministic output
A generated root sheet and project file make the three sheets one
hierarchical KiCad 10 project: 49 connectors, 153 nets. One fewer net than
the sheets separately, because a global label shared between sheets now
joins them - the way an off-sheet flag is meant to mean the same net
everywhere.

UUIDs are now derived deterministically instead of drawn at random. A
generated file under version control that changed every UUID on every
regeneration would show every line modified each time, burying the real
differences. Regenerating an unchanged wire list is now byte-identical.

Reference designators are prefixed per sheet (J101, J201, ...) so they are
unique across the project, and each symbol carries both a standalone and a
hierarchical instance path, so every sheet still verifies on its own and
annotates cleanly inside the project.

Co-Authored-By: Claude Opus 5.5 <noreply@anthropic.com>
Claude-Session: https://claude.ai/code/session_015SpGdnvPFhutgEDurpngu2
Parts:
- removed J1: VP-X J2, symbol n720ak:VP-X_J2
- removed J10: ALTERNATOR, symbol n720ak:ALTERNATOR
- removed J11: KEYSWITCH, symbol n720ak:KEYSWITCH
- removed J12: ENGINE START, symbol n720ak:ENGINE_START
- removed J13: ANN ECU PWR PRI (GRN), symbol n720ak:ANN_ECU_PWR_PRI__GRN_
- removed J14: ANN ECU PWR SEC (GRN), symbol n720ak:ANN_ECU_PWR_SEC__GRN_
- removed J15: ANN FUEL PUMP 1 (GRN), symbol n720ak:ANN_FUEL_PUMP_1__GRN_
- removed J16: ANN FUEL PUMP 2 (AMB), symbol n720ak:ANN_FUEL_PUMP_2__AMB_
- removed J17: ANN ECU FAULT PRI (RED), symbol n720ak:ANN_ECU_FAULT_PRI__RED_
- removed J18: ANN ECU FAULT SEC (RED), symbol n720ak:ANN_ECU_FAULT_SEC__RED_
- removed J19: PILOT-SW-PANEL DB15, symbol n720ak:PILOT-SW-PANEL_DB15
- removed J2: COPILOT-SW-PANEL DB15, symbol n720ak:COPILOT-SW-PANEL_DB15
- removed J20: START CONTACTOR 1, symbol n720ak:START_CONTACTOR_1
- removed J21: START CONTACTOR 2, symbol n720ak:START_CONTACTOR_2
- removed J22: FUEL PUMP CHANGEOVER RELAY, symbol n720ak:FUEL_PUMP_CHANGEOVER_RELAY
- removed J23: FUEL PUMP MODE, symbol n720ak:FUEL_PUMP_MODE
- removed J24: START BAT SEL, symbol n720ak:START_BAT_SEL
- removed J3: VP-X J1, symbol n720ak:VP-X_J1
- removed J4: VP-X J12, symbol n720ak:VP-X_J12
- removed J5: VP-X J10, symbol n720ak:VP-X_J10
- removed J6: ESS BUS, symbol n720ak:ESS_BUS
- removed J7: BATT 1, symbol n720ak:BATT_1
- removed J8: BATT 2, symbol n720ak:BATT_2
- removed J9: BUS MANAGER, symbol n720ak:BUS_MANAGER
- added J101: VP-X J2, symbol n720ak:VP-X_J2
- added J102: COPILOT-SW-PANEL DB15, symbol n720ak:COPILOT-SW-PANEL_DB15
- added J103: VP-X J1, symbol n720ak:VP-X_J1
- added J104: VP-X J12, symbol n720ak:VP-X_J12
- added J105: VP-X J10, symbol n720ak:VP-X_J10
- added J106: ESS BUS, symbol n720ak:ESS_BUS
- added J107: BATT 1, symbol n720ak:BATT_1
- added J108: BATT 2, symbol n720ak:BATT_2
- added J109: BUS MANAGER, symbol n720ak:BUS_MANAGER
- added J110: ALTERNATOR, symbol n720ak:ALTERNATOR
- added J111: KEYSWITCH, symbol n720ak:KEYSWITCH
- added J112: ENGINE START, symbol n720ak:ENGINE_START
- added J113: ANN ECU PWR PRI (GRN), symbol n720ak:ANN_ECU_PWR_PRI__GRN_
- added J114: ANN ECU PWR SEC (GRN), symbol n720ak:ANN_ECU_PWR_SEC__GRN_
- added J115: ANN FUEL PUMP 1 (GRN), symbol n720ak:ANN_FUEL_PUMP_1__GRN_
- added J116: ANN FUEL PUMP 2 (AMB), symbol n720ak:ANN_FUEL_PUMP_2__AMB_
- added J117: ANN ECU FAULT PRI (RED), symbol n720ak:ANN_ECU_FAULT_PRI__RED_
- added J118: ANN ECU FAULT SEC (RED), symbol n720ak:ANN_ECU_FAULT_SEC__RED_
- added J119: PILOT-SW-PANEL DB15, symbol n720ak:PILOT-SW-PANEL_DB15
- added J120: START CONTACTOR 1, symbol n720ak:START_CONTACTOR_1
- added J121: START CONTACTOR 2, symbol n720ak:START_CONTACTOR_2
- added J122: FUEL PUMP CHANGEOVER RELAY, symbol n720ak:FUEL_PUMP_CHANGEOVER_RELAY
- added J123: FUEL PUMP MODE, symbol n720ak:FUEL_PUMP_MODE
- added J124: START BAT SEL, symbol n720ak:START_BAT_SEL
Connections:
- net A/P SERVO POWER: now also J119.5
- net AG: now also J102.1, J102.4, J102.6, J104.4, J105.9, J109.GND, J113.2, J114.2, J115.2, J116.2, J119.1, J119.9
- net AIRFRAME GROUND: now also J107.-, J108.-
- net ALT CURRENT LIMITER: now also J107.+, J109.Batt1/Alt, J110.B, J120.BAT
- net ALT FIELD SWITCH: now also J110.FIELD
- net ALTERNATOR FIELD: now also J106.ALT_FLD
- net BOSE JACKS Pin 1: now also J105.4
- net CABIN LIGHTS POWER: now also J105.3
- net CO DETECT J1-1: now also J105.8
- net COM RELAY 30: now also J106.COM_1
- net DEFROST FAN PWR: now also J103.1
- net ECU CHECK ENG PRI: now also J117.2
- net ECU CHECK ENG SEC: now also J118.2
- net EFIS (ALL) SERIAL 1: now also J103.20, J103.22
- net EMERG POWER SWITCH: now also J109.E-Pwr-1, J109.E-Pwr-2
- net ESSENTIAL BUS BAR: now also J109.Essential_Bus_Pwr, J112.4, J123.2, J124.2
- net ETHERNET SWITCH: now also J104.9
- net FLAP MOTOR: now also J104.5, J104.6
- net FLAP POSITION SENSOR: now also J103.17, J103.18, J103.19
- net FLAPS SWITCH: now also J101.14, J101.15
- net FUEL PRESS INPUT: now also J109.top_harness, J122.85
- net FUEL PUMP 1 PWR: now also J106.PUMP_1
- net FUEL PUMP 2 PWR: now also J106.PUMP_2
- net IGNITION PWR: now also J106.IGN_PWR
- net LANDING LIGHTS POWER: now also J104.1
- net LEFT MAP LT: now also J102.10, J102.9
- net MH OXYGEN CONTROL HEAD: now also J102.13
- net NAV LIGHTS POWER: now also J105.5
- net NAV RELAY 30: now also J106.NAV_1
- net PANEL LED STRIP - PLUS: now also J102.8
- net PITOT HEAT POWER: now also J105.6
- net PLX AIR/FUEL MODULE: now also J105.10
- net PRIMARY ECU PWR: now also J106.ECU_PRI
- net RIGHT MAP LT: now also J102.11, J102.12
- net SECONDARY ECU PWR: now also J106.ECU_SEC
- net STARTER: now also J120.OUT, J121.OUT
- net STARTER CONTACTOR: now also J101.11
- net STROBE LIGHTS POWER: now also J104.2
- net SV-A/P-PNL D15-9: now also J104.10
- net SV-ADSB-470 J1-1: now also J105.7
- net SV-COM D15-8: now also J104.7
- net SV-HDX1100 (PFD) D37-1/20: now also J106.PFD
- net SV-HDX1100 (PFD2) D37-1/20: now also J105.2
- net TAXI LIGHTS POWER: now also J104.3
- net USB CHARGERS: now also J104.8
- net VP-X SPORT: now also J109.Main_Bus_Pwr
- net WIGWAG POWER: now also J104.12
- new net: J101.5, J119.11
- new net: J101.6, J119.12
- new net: J101.7, J119.13
- new net: J101.1, J119.2
- new net: J101.2, J119.6
- new net: J101.3, J119.7
- new net: J101.4, J119.8
- new net: J109.left_harness, J111.1, J111.3, J112.3
- new net: J108.+, J109.Batt_2, J121.BAT
- new net: J109.bottom_harness, J123.1, J123.3, J124.1, J124.3
- new net: J101.8, J102.2
- new net: J101.9, J102.3

Commit message: Record modifications since 2017 and draw the airplane as built
The SteinAir drawings date from 2017. Adds wiring/changes.tsv, a numbered,
dated record of each modification since, and scripts/wirelist_changes.py,
which applies them to the as-drawn wire lists to produce as-built lists in
wiring/as-built/. The KiCad sheets are now drawn from the as-built lists.

First eleven changes, from the owner:

- SV-ADSB-470 swapped for the 472 (2019-04-02); box swap, wiring unchanged.
- The GTN's RS-232 port 4 cut from SkyView Serial 4. Serial 4 TX now feeds
  OnSpeed; Serial 4 RX is unused.
- CO detector audio removed from GMA 245 J1-29; OnSpeed audio took its
  place.
- OnSpeed and the front USB-C charger each fed from the essential bus
  through a discrete fuse.
- MZ-30 current output on EMS pin 31, where the CO detector's EMS output
  used to be. The MZ-30 status wire is not connected.

Removing a pin from a net needed care. Wire lists store a net as a star
from one pin, so deleting the GTN's rows naively would have split the three
displays' Serial 4 pins apart. "disconnect" re-joins the rest of the net.
A change that matches nothing stops the build rather than silently drawing
the old wiring.

Also verified against the drawing, as the owner asked: all ten serial pins
are tied across all three displays.

Corrects sys-24 from the drawing: VP-X J12-11 (FIELD PRI) is not wired -
the alternator field comes from the essential bus ALT FLD breaker; the
SERVOS breaker is 5 A; wigwag is J12-12; defrost and fault annunciator are
J1-1 and J1-2.

Ignores KiCad's local .kicad_prl state file, which had been committed.

Co-Authored-By: Claude Opus 5.5 <noreply@anthropic.com>
Claude-Session: https://claude.ai/code/session_015SpGdnvPFhutgEDurpngu2
Connections:
- net SV-ADSB-470 J1-1 renamed SV-ADSB-472 J1-1
Other:
- note added: "Red 5A"
Changed lines of the file:
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@@
 	(generator "n720ak_kicad_harness")
 	(generator_version "10.0")
-	(paper "User" 420 496)
+	(paper "User" 420 517)
 	(title_block (title "Power & Lighting") (company "N720AK -- Van's RV-10") (comment 1 "Generated from wiring/PWR.tsv -- edit the wire list, not this sheet"))
 	(symbol (lib_id "n720ak:VP-X_J2") (at 50.8 57.15 0) (unit 1)
@@
 			(path "/16abb5c2-a13d-5411-ba46-47e04cc4479d" (reference "J124") (unit 1))
 			(path "/05ae3897-9dd7-5bc2-b238-7f217081554a/73017f24-3a11-5879-901c-ae364a2c7298" (reference "J124") (unit 1)))))
+	(wire (pts (xy 71.12 452.12) (xy 111.76 452.12)) (stroke (width 0) (type default)))
 	(wire (pts (xy 60.96 43.18) (xy 106.68 43.18)) (stroke (width 0) (type default)))
 	(wire (pts (xy 106.68 43.18) (xy 106.68 44.45)) (stroke (width 0) (type default)))
@@
 	(junction (at 152.4 314.96) (diameter 0) (color 0 0 0 0))
 	(junction (at 154.94 314.96) (diameter 0) (color 0 0 0 0))
+	(global_label "ESSENTIAL BUS BAR" (shape bidirectional) (at 71.12 452.12 180)
+		(effects (font (size 1.27 1.27)) (justify right)))
+	(global_label "FRONT USB-C CHARGER" (shape bidirectional) (at 111.76 452.12 0)
+		(effects (font (size 1.27 1.27)) (justify left)))
 	(global_label "STARTER CONTACTOR" (shape bidirectional) (at 71.12 66.04 0)
 		(effects (font (size 1.27 1.27)) (justify left)))
@@
 	(global_label "SV-XPNDR-261 J1-15" (shape bidirectional) (at 71.12 203.2 0)
 		(effects (font (size 1.27 1.27)) (justify left)))
-	(global_label "SV-ADSB-470 J1-1" (shape bidirectional) (at 71.12 205.74 0)
+	(global_label "SV-ADSB-472 J1-1" (shape bidirectional) (at 71.12 205.74 0)
 		(effects (font (size 1.27 1.27)) (justify left)))
 	(global_label "MH CNTRL HEAD J1-1" (shape bidirectional) (at 71.12 208.28 0)
@@
 	(global_label "ECU CHECK ENG SEC" (shape bidirectional) (at 71.12 436.88 0)
 		(effects (font (size 1.27 1.27)) (justify left)))
+	(text "Red 5A" (at 73.66 452.12 0) (effects (font (size 1.0 1.0)) (justify left bottom)))
 	(text "Vio" (at 63.5 43.18 0) (effects (font (size 1.0 1.0)) (justify left bottom)))
 	(text "Vio/Blu" (at 63.5 45.72 0) (effects (font (size 1.0 1.0)) (justify left bottom)))

Commit message: Record the owner's second round of answers; add OnSpeed and EMS sheets
24 recorded changes now, from the owner:

- OnSpeed is a Gen2v4 box on a DB-25 harness. Its pinout in sys-34 matches
  Phil's Gen2v4 aircraft harness drawing pin for pin, so the as-installed
  harness gets its own sheet: power from the essential bus through a 1 A
  blade fuse, SkyView Serial 4 TX in, right audio channel as mono into GMA
  245 Alert 3, flap position spliced into the VP-X flap sensor wire, and
  the button, LED and volume pot on a 6-conductor control cable.
- The CO detector is installed and powered. Only its audio and EMS data
  wires were cut - the audio input now carries OnSpeed and the EMS pin
  carries the MZ-30. sys-42 said it was not installed; corrected.
- EMS pin 31 is on the DB37 - the EMS's other connector has only 25 pins.
- COM 2 flip/flop has been wired to the grips since the build; the 2017
  drawing omits it. Recorded, with its return pin still to confirm.
- The GTN serial cut, OnSpeed, USB and MZ-30 work dates to about February
  2026.

Cross-sheet references follow the SteinAir convention: each sheet names
the far end as a label (ONSPEED DB25-10 on one side, GMA245 J1-29 on the
other).

sys-34 corrected: OnSpeed audio goes straight to the GMA 245, not through
the SkyView; power is from the essential bus on 1 A, not from the PFD on
2 A; the left audio channel is unused.

Five sheets, all verifying clean against their as-built wire lists.

Co-Authored-By: Claude Opus 5.5 <noreply@anthropic.com>
Claude-Session: https://claude.ai/code/session_015SpGdnvPFhutgEDurpngu2
Other:
- note added: "Red 1A"
- moved on the sheet: J104, J105, J106, J107, J108, J109, J110, J111, J112, J113, J114, J115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

Commit message: Trace the power sheet's long runs; verify hand-entered wiring against the drawing
The power sheet goes from 18 flagged rows to 1. The line tracer now
settles what was read by eye:

- Pilot DB15-3 (AV MSTR) reaches pin 85 of both GTN power relay coils;
  pilot DB15-4 reaches the ESS SERVOS breaker; copilot DB15-7 reaches ESS
  PNL LTS, and inside the panel powers all four LED dimmers.
- Pilot DB15-10 and copilot DB15-5 are one wire: switch backlighting from
  the SWITCHES dimmer. The earlier transcription had sent both to the
  annunciator, which was wrong.
- The annunciator is a diode-OR lamp test, now drawn as real parts. Each
  power lamp's anode is fed from its essential-bus breaker through D1-D4
  and from the test bus through D5-D8. The test button is two-pole: pole 1
  connects VP-X J1-2 (the second, Yel, line on that pin) to the test bus;
  pole 2 grounds the FAULT lamp cathodes through D9/D10. The earlier
  transcription ran lamp anodes straight to the breakers, skipping the
  diodes.
- The Bus Manager's Blk 16 ga wire feeds Start Contactor 1's coil and Red
  feeds Contactor 2; Pur goes to FUEL PRESS INPUT; Gray to the pump
  changeover relay coil.

Every hand-entered connection on this sheet is now a check: extraction
fails unless the tracer finds it in the drawing's geometry. 31 connection
checks and 3 separation checks, including that the test button's contacts
are open.

Two tracer bugs found by those checks, both of which silently cut real
wires:

- Lines drawn 0.2-1.3 degrees off vertical were discarded as diagonals,
  breaking the FUEL PUMP 2 and ECU FAULT SEC lamp wires. Real diagonals on
  these sheets are all 4 degrees or more; within 3 is now a wire.
- Vertical lines were indexed by their starting y instead of their x, so a
  wire ending partway along one was not seen to touch it. Fixing it changed
  nothing on the other sheets.

Adds wiring/INSPECT.md, a generated condition-inspection checklist of
everything the drawings cannot settle and every c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
Parts:
- added J125: START BAT SEL, symbol n720ak:START_BAT_SEL
- added J126: ANN ECU PWR PRI, symbol n720ak:ANN_ECU_PWR_PRI
- added J127: D5, symbol n720ak:D5
- added J128: ANN ECU PWR SEC, symbol n720ak:ANN_ECU_PWR_SEC
- added J129: D6, symbol n720ak:D6
- added J130: ANN FUEL PUMP 1, symbol n720ak:ANN_FUEL_PUMP_1
- added J131: D7, symbol n720ak:D7
- added J132: ANN FUEL PUMP 2, symbol n720ak:ANN_FUEL_PUMP_2
- added J133: D8, symbol n720ak:D8
- added J134: D9, symbol n720ak:D9
- added J135: D10, symbol n720ak:D10
- J104: value VP-X J12 -> ANN ECU FAULT PRI; symbol n720ak:VP-X_J12 -> n720ak:ANN_ECU_FAULT_PRI
- J105: value VP-X J10 -> ANN ECU FAULT SEC; symbol n720ak:VP-X_J10 -> n720ak:ANN_ECU_FAULT_SEC
- J106: value ESS BUS -> ANN LT TEST; symbol n720ak:ESS_BUS -> n720ak:ANN_LT_TEST
- J107: value BATT 1 -> VP-X J12; symbol n720ak:BATT_1 -> n720ak:VP-X_J12
- J108: value BATT 2 -> VP-X J10; symbol n720ak:BATT_2 -> n720ak:VP-X_J10
- J109: value BUS MANAGER -> ESS BUS; symbol n720ak:BUS_MANAGER -> n720ak:ESS_BUS
- J110: value ALTERNATOR -> BATT 1; symbol n720ak:ALTERNATOR -> n720ak:BATT_1
- J111: value KEYSWITCH -> BATT 2; symbol n720ak:KEYSWITCH -> n720ak:BATT_2
- J112: value ENGINE START -> BUS MANAGER; symbol n720ak:ENGINE_START -> n720ak:BUS_MANAGER
- J113: value ANN ECU PWR PRI (GRN) -> ALTERNATOR; symbol n720ak:ANN_ECU_PWR_PRI__GRN_ -> n720ak:ALTERNATOR
- J114: value ANN ECU PWR SEC (GRN) -> KEYSWITCH; symbol n720ak:ANN_ECU_PWR_SEC__GRN_ -> n720ak:KEYSWITCH
- J115: value ANN FUEL PUMP 1 (GRN) -> ENGINE START; symbol n720ak:ANN_FUEL_PUMP_1__GRN_ -> n720ak:ENGINE_START
- J116: value ANN FUEL PUMP 2 (AMB) -> PILOT-SW-PANEL DB15; symbol n720ak:ANN_FUEL_PUMP_2__AMB_ -> n720ak:PILOT-SW-PANEL_DB15
- J117: value ANN ECU FAULT PRI (RED) -> D1; symbol n720ak:ANN_ECU_FAULT_PRI__RED_ -> n720ak:D1
- J118: value ANN ECU FAULT SEC (RED) -> D2; symbol n720ak:ANN_ECU_FAULT_SEC__RED_ -> n720ak:D2
- J119: value PILOT-SW-PANEL DB15 -> D3; symbol n720ak:PILOT-SW-PANEL_DB15 -> n720ak:D3
- J120: value START CONTACTOR 1 -> D4; symbol n720ak:START_CONTACTOR_1 -> n720ak:D4
- J121: value START CONTACTOR 2 -> START CONTACTOR 1; symbol n720ak:START_CONTACTOR_2 -> n720ak:START_CONTACTOR_1
- J122: value FUEL PUMP CHANGEOVER RELAY -> START CONTACTOR 2; symbol n720ak:FUEL_PUMP_CHANGEOVER_RELAY -> n720ak:START_CONTACTOR_2
- J123: value FUEL PUMP MODE -> FUEL PUMP CHANGEOVER RELAY; symbol n720ak:FUEL_PUMP_MODE -> n720ak:FUEL_PUMP_CHANGEOVER_RELAY
- J124: value START BAT SEL -> FUEL PUMP MODE; symbol n720ak:START_BAT_SEL -> n720ak:FUEL_PUMP_MODE
Connections:
- net A/P SERVO POWER: now also J116.5; no longer J119.5
- net AG: now also J106.2B, J107.4, J108.9, J112.GND, J116.1, J116.9, J126.2, J128.2, J130.2, J132.2; no longer J104.4, J105.9, J109.GND, J113.2, J114.2, J115.2, J116.2, J119.1, J119.9
- net AIRFRAME GROUND: now also J110.-, J111.-; no longer J107.-, J108.-
- net ALT CURRENT LIMITER: now also J110.+, J112.Batt1/Alt, J113.B, J121.BAT; no longer J107.+, J109.Batt1/Alt, J110.B, J120.BAT
- net ALT FIELD SWITCH: now also J113.FIELD; no longer J110.FIELD
- net ALTERNATOR FIELD: now also J109.ALT_FLD; no longer J106.ALT_FLD
- net BOSE JACKS Pin 1: now also J108.4; no longer J105.4
- net CABIN LIGHTS POWER: now also J108.3; no longer J105.3
- net CO DETECT J1-1: now also J108.8; no longer J105.8
- net COM RELAY 30: now also J109.COM_1; no longer J106.COM_1
- net ECU CHECK ENG PRI: now also J104.2, J134.A; no longer J117.2
- net ECU CHECK ENG SEC: now also J105.2, J135.A; no longer J118.2
- net EMERG POWER SWITCH: now also J112.E-Pwr-1, J112.E-Pwr-2; no longer J109.E-Pwr-1, J109.E-Pwr-2
- net ESSENTIAL BUS BAR: now also J112.Essential_Bus_Pwr, J115.4, J125.2; no longer J109.Essential_Bus_Pwr, J112.4, J123.2
- net ETHERNET SWITCH: now also J107.9; no longer J104.9
- net FLAP MOTOR: now also J107.5, J107.6; no longer J104.5, J104.6
- net FUEL PRESS INPUT: now also J112.top_harness, J121.coil, J122.coil, J123.85; no longer J109.top_harness, J122.85
- net FUEL PUMP 1 PWR: now also J109.PUMP_1, J119.A; no longer J106.PUMP_1
- net FUEL PUMP 2 PWR: now also J109.PUMP_2, J120.A; no longer J106.PUMP_2
- net IGNITION PWR: now also J109.IGN_PWR; no longer J106.IGN_PWR
- net LANDING LIGHTS POWER: now also J107.1; no longer J104.1
- net NAV LIGHTS POWER: now also J108.5; no longer J105.5
- net NAV RELAY 30: now also J109.NAV_1; no longer J106.NAV_1
- net PITOT HEAT POWER: now also J108.6; no longer J105.6
- net PLX AIR/FUEL MODULE: now also J108.10; no longer J105.10
- net PRIMARY ECU PWR: now also J109.ECU_PRI, J117.A; no longer J106.ECU_PRI
- net SECONDARY ECU PWR: now also J109.ECU_SEC, J118.A; no longer J106.ECU_SEC
- net STARTER: now also J122.OUT; no longer J120.OUT
- net STROBE LIGHTS POWER: now also J107.2; no longer J104.2
- net SV-A/P-PNL D15-9: now also J107.10; no longer J104.10
- net SV-ADSB-472 J1-1: now also J108.7; no longer J105.7
- net SV-COM D15-8: now also J107.7; no longer J104.7
- net SV-HDX1100 (PFD) D37-1/20: now also J109.PFD; no longer J106.PFD
- net SV-HDX1100 (PFD2) D37-1/20: now also J108.2; no longer J105.2
- net TAXI LIGHTS POWER: now also J107.3; no longer J104.3
- net USB CHARGERS: now also J107.8; no longer J104.8
- net VP-X SPORT: now also J112.Main_Bus_Pwr; no longer J109.Main_Bus_Pwr
- net WIGWAG POWER: now also J107.12; no longer J104.12
- net at J101.5: now also J116.11; no longer J119.11
- net at J101.6: now also J116.12; no longer J119.12
- net at J101.7: now also J116.13; no longer J119.13
- net at J101.1: now also J116.2; no longer J119.2
- net at J101.2: now also J116.6; no longer J119.6
- net at J101.3: now also J116.7; no longer J119.7
- net at J101.4: now also J116.8; no longer J119.8
- new net: J118.K, J128.1, J129.K
- new net: J119.K, J130.1, J131.K
- new net: J103.2, J104.1, J105.1, J106.1A
- new net: J106.1B, J127.A, J129.A, J131.A, J133.A
- new net: J106.2A, J134.K, J135.K
- new net: J120.K, J132.1, J133.K
- new net: J111.+, J112.Batt_2, J122.BAT
- new net: J112.bottom_harness, J124.1, J124.3, J125.1, J125.3
- new net: J112.left_harness, J114.1, J114.3, J115.3
- new net: J102.5, J116.10
- new net: J102.7, J109.PNL_LTS
- new net: J117.K, J126.1, J127.K
- new net: J109.SERVOS, J116.4
- new net COM/NAV RELAY COILS (85): J116.3
Other:
- note added: "Blk 16 AWG"
- note added: "Wht/Blk"
- note added: "Wht/Ora"
- moved on the sheet: J110, J111, J120, J124
