File: kicad/n720ak/SV.kicad_sch (KiCad schematic)
At the start: 19 parts, among them J1 GMA245 J1, J10 GTN 650 P1003, J11 GTN P1004, J12 MH OXYGEN CONTROL HEAD, J13 Skyview ARINC DB25, J14 R-XPNDR-GPS (1.21 kOhm series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, J15 SV-HDX1100 (PFD - LEFT #1) DB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, J16 SV-HDX800 (MFD – CENTER #2) D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, J17 SV-COM-PANEL DB15, J18 SV-ADSB-470 DB9, J19 VP-X SPORT J1, J2 SV-COM C25 DB15, J3 GTN P1001, J4 CO DETECTOR 452-101-011 DB9, J5 ARTEX 345 ELT DB15, J6 SV-HDX1100 (PFD2 – RIGHT #3) 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, J7 GMA245 J2, J8 SV-XPNDR-261 DB-25M, J9 SV-AP-PANEL DB-15

Commit message: Tie the sheets into one KiCad project with deterministic output
A generated root sheet and project file make the three sheets one
hierarchical KiCad 10 project: 49 connectors, 153 nets. One fewer net than
the sheets separately, because a global label shared between sheets now
joins them - the way an off-sheet flag is meant to mean the same net
everywhere.

UUIDs are now derived deterministically instead of drawn at random. A
generated file under version control that changed every UUID on every
regeneration would show every line modified each time, burying the real
differences. Regenerating an unchanged wire list is now byte-identical.

Reference designators are prefixed per sheet (J101, J201, ...) so they are
unique across the project, and each symbol carries both a standalone and a
hierarchical instance path, so every sheet still verifies on its own and
annotates cleanly inside the project.

Co-Authored-By: Claude Opus 5.5 <noreply@anthropic.com>
Claude-Session: https://claude.ai/code/session_015SpGdnvPFhutgEDurpngu2
Parts:
- removed J1: GMA245 J1, symbol n720ak:GMA245_J1
- removed J10: GTN 650 P1003, symbol n720ak:GTN_650_P1003
- removed J11: GTN P1004, symbol n720ak:GTN_P1004
- removed J12: MH OXYGEN CONTROL HEAD, symbol n720ak:MH_OXYGEN_CONTROL_HEAD
- removed J13: Skyview ARINC DB25, symbol n720ak:Skyview_ARINC_DB25
- removed J14: R-XPNDR-GPS (1.21 kOhm series resistor), symbol n720ak:R-XPNDR-GPS__1.21_kOhm_series_resistor_
- removed J15: SV-HDX1100 (PFD - LEFT #1) DB37, symbol n720ak:SV-HDX1100__PFD_-_LEFT__1__DB37
- removed J16: SV-HDX800 (MFD – CENTER #2) DB37, symbol n720ak:SV-HDX800__MFD___CENTER__2__DB37
- removed J17: SV-COM-PANEL DB15, symbol n720ak:SV-COM-PANEL_DB15
- removed J18: SV-ADSB-470 DB9, symbol n720ak:SV-ADSB-470_DB9
- removed J19: VP-X SPORT J1, symbol n720ak:VP-X_SPORT_J1
- removed J2: SV-COM C25 DB15, symbol n720ak:SV-COM_C25_DB15
- removed J3: GTN P1001, symbol n720ak:GTN_P1001
- removed J4: CO DETECTOR 452-101-011 DB9, symbol n720ak:CO_DETECTOR_452-101-011_DB9
- removed J5: ARTEX 345 ELT DB15, symbol n720ak:ARTEX_345_ELT_DB15
- removed J6: SV-HDX1100 (PFD2 – RIGHT #3) DB37, symbol n720ak:SV-HDX1100__PFD2___RIGHT__3__DB37
- removed J7: GMA245 J2, symbol n720ak:GMA245_J2
- removed J8: SV-XPNDR-261 DB-25M, symbol n720ak:SV-XPNDR-261_DB-25M
- removed J9: SV-AP-PANEL DB-15, symbol n720ak:SV-AP-PANEL_DB-15
- added J201: GMA245 J1, symbol n720ak:GMA245_J1
- added J202: SV-COM C25 DB15, symbol n720ak:SV-COM_C25_DB15
- added J203: GTN P1001, symbol n720ak:GTN_P1001
- added J204: CO DETECTOR 452-101-011 DB9, symbol n720ak:CO_DETECTOR_452-101-011_DB9
- added J205: ARTEX 345 ELT DB15, symbol n720ak:ARTEX_345_ELT_DB15
- added J206: SV-HDX1100 (PFD2 – RIGHT #3) DB37, symbol n720ak:SV-HDX1100__PFD2___RIGHT__3__DB37
- added J207: GMA245 J2, symbol n720ak:GMA245_J2
- added J208: SV-XPNDR-261 DB-25M, symbol n720ak:SV-XPNDR-261_DB-25M
- added J209: SV-AP-PANEL DB-15, symbol n720ak:SV-AP-PANEL_DB-15
- added J210: GTN 650 P1003, symbol n720ak:GTN_650_P1003
- added J211: GTN P1004, symbol n720ak:GTN_P1004
- added J212: MH OXYGEN CONTROL HEAD, symbol n720ak:MH_OXYGEN_CONTROL_HEAD
- added J213: Skyview ARINC DB25, symbol n720ak:Skyview_ARINC_DB25
- added J214: R-XPNDR-GPS (1.21 kOhm series resistor), symbol n720ak:R-XPNDR-GPS__1.21_kOhm_series_resistor_
- added J215: SV-HDX1100 (PFD - LEFT #1) DB37, symbol n720ak:SV-HDX1100__PFD_-_LEFT__1__DB37
- added J216: SV-HDX800 (MFD – CENTER #2) DB37, symbol n720ak:SV-HDX800__MFD___CENTER__2__DB37
- added J217: SV-COM-PANEL DB15, symbol n720ak:SV-COM-PANEL_DB15
- added J218: SV-ADSB-470 DB9, symbol n720ak:SV-ADSB-470_DB9
- added J219: VP-X SPORT J1, symbol n720ak:VP-X_SPORT_J1
Connections:
- net 7 8: now also J205.14 (External On), J205.3 (2-Wire Remote Switch)
- net COPILOT GRIP: now also J209.12 (Copilot Trim Right Button), J209.13 (Copilot Trim Left Button), J209.5 (Copilot Trim Up Button), J209.6 (Copilot Trim Down Button)
- net COPILOT HEADSET JACK (mic): now also J207.32 (Copilot Mic HI), J207.33 (CoPilot Mic PTT)
- net COPILOT HEADSET JACK (phones): now also J207.2 (CoPilot Phones Lo), J207.3 (CoPlilot Phones L), J207.4 (CoPilot Phones R)
- net GROUND: now also J202.12 (GROUND IN), J204.5 (Ground), J205.7 (Ground), J206.21 (GROUND), J206.22 (GROUND), J208.14 (GROUND), J209.2 (Ground -), J213.20 (Ground), J218.4 (Ground)
- net GTN CONFIG MODULE: now also J203.62 (Config Mod Data), J203.65 (Config Mod Power)
- net GTN FAN: now also J203.43 (Fan Ground)
- net PASSENGER HEADSET JACK (mic): now also J207.35 (Pass. Mic Hi), J207.36 (Pass. Mic Lo), J207.37 (Pass. 2 Mic Hi), J207.38 (Pass. 2 Mic Lo)
- net PASSENGER HEADSET JACK (phones): now also J201.40 (Pass. Phone L), J201.41 (Pass. Phones R), J201.42 (Pass. Phone Lo)
- net PILOT GRIP: now also J209.10 (Pilot Trim Right Button), J209.11 (Pilot Trim Left Button), J209.3 (Pilot Trim Up Button), J209.4 (Pilot Trim Down Button)
- net PILOT HEADSET JACK (mic): now also J201.33 (Pilot Mic Hi), J201.34 (Pilot Mic PTT), J201.35 (Pilot Mic Lo)
- net PILOT HEADSET JACK (phones): now also J207.1 (Pilot Phones Lo), J207.16 (Pilot Phones L), J207.31 (Pilot Phones R)
- net SV-GPS-250: now also J206.11 (Serial 5 RX), J206.12 (Serial 5 TX), J206.24 (SV-GPS-250 Ground), J206.29 (SV-GPS-250 Power), J215.11, J215.12, J215.24, J215.29, J216.11, J216.12, J216.24, J216.29
- net USB Socket: now also J206.16 (USB Power), J206.17 (USB Ground (withshield)), J206.18 (USB Data -), J206.19 (USB Data +), J215.16 (USB Power), J215.17 (USB Ground (withshield)), J215.18 (USB Data -), J215.19 (USB Data +), J216.16 (USB Power), J216.17 (USB Ground (withshield)), J216.18 (USB Data -), J216.19 (USB Data +)
- net VP-X J10-2: now also J206.1 (POWER), J206.20
- net VP-X J10-4: now also J207.8 (11-33 VDC), J207.9
- net VP-X J10-7: now also J208.15 (POWER), J218.1 (Power)
- net VP-X J10-8: now also J204.1 (Power)
- net VP-X J12-10: now also J209.9 (Power In +)
- net VP-X J12-7: now also J202.8 (POWER IN)
- net VP-X J12-9: now also J216.1 (POWER), J216.20
- new net: J207.10 (Ground), J207.11
- new net: J206.30, J207.14 (Alert 2 Audio Lo), J215.30, J216.30
- new net: J206.13, J206.31, J207.15 (Alert 2 Audio Hi), J215.13, J215.31, J216.13, J216.31
- new net: J201.10 (Com 1 Lo), J210.18, J210.20
- new net: J201.11 (Com 1 Mic HI), J210.5
- new net: J201.12 (Com 1 Mic Key), J210.11
- new net: J201.13, J202.10 (PHONES OUT)
- new net: J201.14, J202.2 (MIC LO), J202.9
- new net: J201.15, J202.1 (MIC HI)
- new net: J201.17 (Nav 1 Audio Hi), J211.16
- new net: J201.18 (Nav 1 Lo), J211.17
- new net: J201.29 (Alert 3 Audio Hi), J204.6
- new net: J201.30, J202.5 (PTT IN)
- new net: J201.31 (Alert 1 Audio Hi), J203.4
- new net: J201.32 (Alert 1 Audio Lo), J203.23
- new net: J201.44 (Alert 4 Audio Hi), J212.DB25-9
- new net: J201.9 (Com 1 Audio Hi), J210.7
- new net: J206.3 (Serial 1 RX), J215.3, J216.3, J219.20
- new net: J206.4 (Serial 1 TX), J215.4, J216.4, J219.22
- new net: J202.7 (SV-COM POWER), J217.1
- new net: J202.13 (SV COM GROUND), J217.2
- new net: J202.6 (SV-COM-PANEL DATA IN), J217.4
- new net: J202.14 (SV COM DATA OUT), J217.5
- new net: J202.3 (SV COM PANEL ENABLE), J217.6
- new net: J206.6 (Serial 2 TX), J215.6, J216.6, J218.2
- new net: J206.5 (Serial 2 RX), J215.5, J216.5, J218.3
- new net: J205.12, J205.5 (G-Switch Loop)
- new net: J203.6 (GPS RS-232 Out 3), J205.9
- new net: J210.30 (POWER), J210.43, J210.44
- new net: J210.37 (GROUND), J210.38, J210.40
- new net: J211.23 (VOR/ILS Arinc Out B), J213.10
- new net: J203.29 (GPS ARINC 429 OUT 1B), J213.11
- new net: J203.67 (GPS ARINC 429 IN 1B), J213.12
- new net: J211.24 (VOR/ILS Arinc Out A), J213.22
- new net: J203.10 (GPS ARINC 429 OUT 1A), J213.23
- new net: J203.48 (GPS ARINC 429 IN 1A), J213.24
- new net: J203.8 (GPS RS-232 Out 1), J213.3
- new net: J215.1 (POWER), J215.20
- new net: J203.24 (GPS RS-232 In 4), J206.10, J215.10, J216.10
- new net: J215.21 (GROUND), J215.22
- new net: J206.7, J208.7 (Serial Out), J215.7, J216.7
- new net: J206.8, J208.5 (Serial In), J215.8, J216.8
- new net: J203.5 (GPS RS-232 Out 4), J206.9, J215.9, J216.9
- new net: J203.7 (GPS RS-232 Out 2), J214.1
- new net: J208.3 (GPS In (ADS-B)), J214.2
- new net: J203.19 (POWER 1), J203.20, J211.51, J211.52
- new net: J203.77 (GROUND), J203.78, J211.61, J211.62
- new net: J208.1 (Jumper), J208.2
- new net: J208.12 (Jumper), J208.13
- new net: J216.21 (GROUND), J216.22

Commit message: Record modifications since 2017 and draw the airplane as built
The SteinAir drawings date from 2017. Adds wiring/changes.tsv, a numbered,
dated record of each modification since, and scripts/wirelist_changes.py,
which applies them to the as-drawn wire lists to produce as-built lists in
wiring/as-built/. The KiCad sheets are now drawn from the as-built lists.

First eleven changes, from the owner:

- SV-ADSB-470 swapped for the 472 (2019-04-02); box swap, wiring unchanged.
- The GTN's RS-232 port 4 cut from SkyView Serial 4. Serial 4 TX now feeds
  OnSpeed; Serial 4 RX is unused.
- CO detector audio removed from GMA 245 J1-29; OnSpeed audio took its
  place.
- OnSpeed and the front USB-C charger each fed from the essential bus
  through a discrete fuse.
- MZ-30 current output on EMS pin 31, where the CO detector's EMS output
  used to be. The MZ-30 status wire is not connected.

Removing a pin from a net needed care. Wire lists store a net as a star
from one pin, so deleting the GTN's rows naively would have split the three
displays' Serial 4 pins apart. "disconnect" re-joins the rest of the net.
A change that matches nothing stops the build rather than silently drawing
the old wiring.

Also verified against the drawing, as the owner asked: all ten serial pins
are tied across all three displays.

Corrects sys-24 from the drawing: VP-X J12-11 (FIELD PRI) is not wired -
the alternator field comes from the essential bus ALT FLD breaker; the
SERVOS breaker is 5 A; wigwag is J12-12; defrost and fault annunciator are
J1-1 and J1-2.

Ignores KiCad's local .kicad_prl state file, which had been committed.

Co-Authored-By: Claude Opus 5.5 <noreply@anthropic.com>
Claude-Session: https://claude.ai/code/session_015SpGdnvPFhutgEDurpngu2
Parts:
- added J220: ONSPEED, symbol n720ak:ONSPEED
- J204: value CO DETECTOR 452-101-011 DB9 -> ARTEX 345 ELT DB15; symbol n720ak:CO_DETECTOR_452-101-011_DB9 -> n720ak:ARTEX_345_ELT_DB15
- J205: value ARTEX 345 ELT DB15 -> GMA245 J2; symbol n720ak:ARTEX_345_ELT_DB15 -> n720ak:GMA245_J2
- J207: value GMA245 J2 -> SV-XPNDR-261 DB-25M; symbol n720ak:GMA245_J2 -> n720ak:SV-XPNDR-261_DB-25M
- J208: value SV-XPNDR-261 DB-25M -> CO DETECTOR 452-101-011 DB9; symbol n720ak:SV-XPNDR-261_DB-25M -> n720ak:CO_DETECTOR_452-101-011_DB9
- J218: value SV-ADSB-470 DB9 -> SV-ADSB-472 DB9; symbol n720ak:SV-ADSB-470_DB9 -> n720ak:SV-ADSB-472_DB9
Connections:
- net 7 8: now also J204.14 (External On), J204.3 (2-Wire Remote Switch); no longer J205.14 (External On), J205.3 (2-Wire Remote Switch)
- net COPILOT HEADSET JACK (mic): now also J205.32 (Copilot Mic HI), J205.33 (CoPilot Mic PTT); no longer J207.32 (Copilot Mic HI), J207.33 (CoPilot Mic PTT)
- net COPILOT HEADSET JACK (phones): now also J205.2 (CoPilot Phones Lo), J205.3 (CoPlilot Phones L), J205.4 (CoPilot Phones R); no longer J207.2 (CoPilot Phones Lo), J207.3 (CoPlilot Phones L), J207.4 (CoPilot Phones R)
- net GROUND: now also J204.7 (Ground), J207.14 (GROUND), J208.5 (Ground), J220.4 (Ground); no longer J204.5 (Ground), J205.7 (Ground), J208.14 (GROUND)
- net PASSENGER HEADSET JACK (mic): now also J205.35 (Pass. Mic Hi), J205.36 (Pass. Mic Lo), J205.37 (Pass. 2 Mic Hi), J205.38 (Pass. 2 Mic Lo); no longer J207.35 (Pass. Mic Hi), J207.36 (Pass. Mic Lo), J207.37 (Pass. 2 Mic Hi), J207.38 (Pass. 2 Mic Lo)
- net PILOT HEADSET JACK (phones): now also J205.1 (Pilot Phones Lo), J205.16 (Pilot Phones L), J205.31 (Pilot Phones R); no longer J207.1 (Pilot Phones Lo), J207.16 (Pilot Phones L), J207.31 (Pilot Phones R)
- net VP-X J10-4: now also J205.8 (11-33 VDC), J205.9; no longer J207.8 (11-33 VDC), J207.9
- net VP-X J10-7: now also J207.15 (POWER); no longer J208.15 (POWER)
- net VP-X J10-8: now also J208.1 (Power); no longer J204.1 (Power)
- net at J206.30, J215.30, J216.30: now also J205.14 (Alert 2 Audio Lo); no longer J207.14 (Alert 2 Audio Lo)
- net at J206.13, J206.31, J215.13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: now also J205.15 (Alert 2 Audio Hi); no longer J207.15 (Alert 2 Audio Hi)
- net at J203.6 (GPS RS-232 Out 3): now also J204.9; no longer J205.9
- net at J206.10 (GPS RS-232 In 4), J215.10 (Serial 4 TX), J216.10: now also J220.25; no longer J203.24 (GPS RS-232 In 4)
- net at J206.7, J215.7, J216.7: now also J207.7 (Serial Out); no longer J208.7 (Serial Out)
- net at J206.8, J215.8, J216.8: now also J207.5 (Serial In); no longer J208.5 (Serial In)
- net at J206.9 (GPS RS-232 Out 4), J215.9, J216.9: no longer J203.5 (GPS RS-232 Out 4)
- net at J214.2: now also J207.3 (GPS In (ADS-B)); no longer J208.3 (GPS In (ADS-B))
- new net: J207.1 (Jumper), J207.2
- new net: J207.12 (Jumper), J207.13
- new net: J205.10 (Ground), J205.11
- new net: J204.12, J204.5 (G-Switch Loop)
Other:
- moved on the sheet: J202, J209, J210, J211, J212, J213, J214, J216, J217, J218, J219

Commit message: Trace the headset jacks, Bose jacks and grips from the drawing
The SkyView sheet's audio area was the largest gap: jacks, the Bose LEMO
jacks and the grip switches are drawn as symbols, not connector boxes, so
the earlier extraction guessed each pin's destination from its name. That
sent the pilot PTT line only to the mic jack, missing the grip, and lost
both Bose jacks entirely.

The tracer now reads them as parts:

- Headset jacks. Their contacts are WHITE filled circles; junction dots are
  BLACK. The two had been confused, so jack contacts were being counted as
  junctions. Contacts are grouped three to a jack as tip, ring and sleeve,
  and jacks are named from the GMA 245 function on their tip.
- Bose LEMO jacks, read as pin columns with a free-text title. Both draw
  power from VP-X J10-4 alongside the GMA 245.
- Grips, read as devices from their dashed outlines. A wire ending inside
  lands on the button whose label sits directly above it - "nearest label"
  picked the next button down.

Fixed on the way, each of which had silently disconnected a real wire:

- The drawing leaves sub-point gaps at some corners (683.4 against 684.0).
  Coordinates are snapped per axis; snapping points moved whole vertical
  lines sideways and broke their other ends.
- Many strokes are drawn two or three times. Duplicates made a wire's loose
  end look like a meeting of two lines, so the grip was never attached.

Grounds that were defaulted to GROUND now trace to the AG symbol, matching
the power sheet. The SkyView sheet goes from 19 flagged rows to 3, all of
them placeholders for regions not yet extracted.

Co-Authored-By: Claude Opus 5.5 <noreply@anthropic.com>
Claude-Session: https://claude.ai/code/session_015SpGdnvPFhutgEDurpngu2
Parts:
- added J221: PILOT PHONE JACK, symbol n720ak:PILOT_PHONE_JACK
- added J222: COPILOT PHONE JACK, symbol n720ak:COPILOT_PHONE_JACK
- added J223: COPILOT BOSE, symbol n720ak:COPILOT_BOSE
- added J224: PASSENGER MIC JACK 1, symbol n720ak:PASSENGER_MIC_JACK_1
- added J225: PASSENGER MIC JACK 2, symbol n720ak:PASSENGER_MIC_JACK_2
- added J226: COPILOT MIC JACK, symbol n720ak:COPILOT_MIC_JACK
- added J227: COPILOT GRIP, symbol n720ak:COPILOT_GRIP
- added J228: SV-HDX1100 (PFD - LEFT #1) DB37, symbol n720ak:SV-HDX1100__PFD_-_LEFT__1__DB37
- added J229: SV-HDX800 (MFD – CENTER #2) DB37, symbol n720ak:SV-HDX800__MFD___CENTER__2__DB37
- added J230: SV-COM-PANEL DB15, symbol n720ak:SV-COM-PANEL_DB15
- added J231: SV-ADSB-472 DB9, symbol n720ak:SV-ADSB-472_DB9
- added J232: VP-X SPORT J1, symbol n720ak:VP-X_SPORT_J1
- added J233: PITCH TRIM SERVO MOTOR, symbol n720ak:PITCH_TRIM_SERVO_MOTOR
- added J234: ROLL TRIM SERVO MOTOR, symbol n720ak:ROLL_TRIM_SERVO_MOTOR
- added J235: ONSPEED, symbol n720ak:ONSPEED
- J210: value GTN 650 P1003 -> PILOT MIC JACK; symbol n720ak:GTN_650_P1003 -> n720ak:PILOT_MIC_JACK
- J211: value GTN P1004 -> PILOT BOSE; symbol n720ak:GTN_P1004 -> n720ak:PILOT_BOSE
- J212: value MH OXYGEN CONTROL HEAD -> PILOT GRIP; symbol n720ak:MH_OXYGEN_CONTROL_HEAD -> n720ak:PILOT_GRIP
- J213: value Skyview ARINC DB25 -> PASSENGER PHONE JACK 1; symbol n720ak:Skyview_ARINC_DB25 -> n720ak:PASSENGER_PHONE_JACK_1
- J214: value R-XPNDR-GPS (1.21 kOhm series resistor) -> PASSENGER PHONE JACK 2; symbol n720ak:R-XPNDR-GPS__1.21_kOhm_series_resistor_ -> n720ak:PASSENGER_PHONE_JACK_2
- J215: value SV-HDX1100 (PFD - LEFT #1) DB37 -> GTN 650 P1003; symbol n720ak:SV-HDX1100__PFD_-_LEFT__1__DB37 -> n720ak:GTN_650_P1003
- J216: value SV-HDX800 (MFD – CENTER #2) DB37 -> GTN P1004; symbol n720ak:SV-HDX800__MFD___CENTER__2__DB37 -> n720ak:GTN_P1004
- J217: value SV-COM-PANEL DB15 -> MH OXYGEN CONTROL HEAD; symbol n720ak:SV-COM-PANEL_DB15 -> n720ak:MH_OXYGEN_CONTROL_HEAD
- J218: value SV-ADSB-472 DB9 -> GRIPS; symbol n720ak:SV-ADSB-472_DB9 -> n720ak:GRIPS
- J219: value VP-X SPORT J1 -> Skyview ARINC DB25; symbol n720ak:VP-X_SPORT_J1 -> n720ak:Skyview_ARINC_DB25
- J220: value ONSPEED -> R-XPNDR-GPS (1.21 kOhm series resistor); symbol n720ak:ONSPEED -> n720ak:R-XPNDR-GPS__1.21_kOhm_series_resistor_
Connections:
- net GROUND: now also J235.4 (Ground); no longer J202.12 (GROUND IN), J206.21 (GROUND), J207.14 (GROUND), J208.5 (Ground), J209.2 (Ground -), J213.20 (Ground), J218.4 (Ground), J220.4 (Ground)
- net GTN CONFIG MODULE: now also J203.63 (Config Mod Clock), J203.64 (Config Mod Ground)
- net GTN FAN: now also J203.58 (Fan Tach In), J203.59 (Fan Power)
- net SV-GPS-250: now also J228.11, J228.12, J228.24, J228.29, J229.11, J229.12, J229.24, J229.29; no longer J215.11, J215.12, J215.24, J215.29, J216.11, J216.12, J216.24, J216.29
- net USB Socket: now also J228.16 (USB Power), J228.17 (USB Ground (withshield)), J228.18 (USB Data -), J228.19 (USB Data +), J229.16 (USB Power), J229.17 (USB Ground (withshield)), J229.18 (USB Data -), J229.19 (USB Data +); no longer J215.16 (USB Power), J215.17 (USB Ground (withshield)), J215.18 (USB Data -), J215.19 (USB Data +), J216.16 (USB Power), J216.17 (USB Ground (withshield)), J216.18 (USB Data -), J216.19 (USB Data +)
- net VP-X J10-4: now also J211.1, J223.1
- net VP-X J10-7: now also J231.1 (Power); no longer J218.1 (Power)
- net VP-X J12-9: now also J229.1 (POWER), J229.20; no longer J216.1 (POWER), J216.20
- net at J207.3 (GPS In (ADS-B)): now also J220.2; no longer J214.2
- net at J206.8, J207.5 (Serial In): now also J228.8, J229.8; no longer J215.8, J216.8
- net at J206.7, J207.7 (Serial Out): now also J228.7, J229.7; no longer J215.7, J216.7
- net at J201.11 (Com 1 Mic HI): now also J215.5; no longer J210.5
- net at J201.12 (Com 1 Mic Key): now also J215.11; no longer J210.11
- net at J201.17 (Nav 1 Audio Hi): now also J216.16; no longer J211.16
- net at J201.18 (Nav 1 Lo): now also J216.17; no longer J211.17
- net at J201.44 (Alert 4 Audio Hi): now also J217.DB25-9; no longer J212.DB25-9
- net at J201.9 (Com 1 Audio Hi): now also J215.7; no longer J210.7
- net at J202.7 (SV-COM POWER): now also J230.1; no longer J217.1
- net at J202.13 (SV COM GROUND): now also J230.2; no longer J217.2
- net at J202.6 (SV-COM-PANEL DATA IN): now also J230.4; no longer J217.4
- net at J202.14 (SV COM DATA OUT): now also J230.5; no longer J217.5
- net at J202.3 (SV COM PANEL ENABLE): now also J230.6; no longer J217.6
- net at J205.14 (Alert 2 Audio Lo), J206.30: now also J228.30, J229.30; no longer J215.30, J216.30
- net at J203.29 (GPS ARINC 429 OUT 1B): now also J219.11; no longer J213.11
- net at J203.67 (GPS ARINC 429 IN 1B): now also J219.12; no longer J213.12
- net at J203.10 (GPS ARINC 429 OUT 1A): now also J219.23; no longer J213.23
- net at J203.48 (GPS ARINC 429 IN 1A): now also J219.24; no longer J213.24
- net at J203.8 (GPS RS-232 Out 1): now also J219.3; no longer J213.3
- net at J215.20: now also J201.10 (Com 1 Lo), J215.18; no longer J215.1 (POWER)
- net at J203.7 (GPS RS-232 Out 2): now also J220.1; no longer J214.1
- net at J203.19 (POWER 1), J203.20: now also J216.51, J216.52; no longer J211.51, J211.52
- net at J203.77 (GROUND), J203.78: now also J216.61, J216.62; no longer J211.61, J211.62
- removed net COPILOT GRIP: J209.12 (Copilot Trim Right Button), J209.13 (Copilot Trim Left Button), J209.5 (Copilot Trim Up Button), J209.6 (Copilot Trim Down Button)
- net COPILOT HEADSET JACK (mic): no longer names the net of J205.33 (CoPilot Mic PTT)
- net COPILOT HEADSET JACK (mic): now also J226.R, J227.PTT-1; no longer J205.32 (Copilot Mic HI)
- removed net COPILOT HEADSET JACK (phones): J205.2 (CoPilot Phones Lo), J205.3 (CoPlilot Phones L), J205.4 (CoPilot Phones R)
- removed net PASSENGER HEADSET JACK (mic): J205.35 (Pass. Mic Hi), J205.36 (Pass. Mic Lo), J205.37 (Pass. 2 Mic Hi), J205.38 (Pass. 2 Mic Lo)
- removed net PASSENGER HEADSET JACK (phones): J201.40 (Pass. Phone L), J201.41 (Pass. Phones R), J201.42 (Pass. Phone Lo)
- removed net PILOT GRIP: J209.10 (Pilot Trim Right Button), J209.11 (Pilot Trim Left Button), J209.3 (Pilot Trim Up Button), J209.4 (Pilot Trim Down Button)
- removed net PILOT HEADSET JACK (mic): J201.33 (Pilot Mic Hi), J201.34 (Pilot Mic PTT), J201.35 (Pilot Mic Lo)
- removed net PILOT HEADSET JACK (phones): J205.1 (Pilot Phones Lo), J205.16 (Pilot Phones L), J205.31 (Pilot Phones R)
- new net: J201.33 (Pilot Mic Hi), J210.T, J211.5
- new net: J201.34 (Pilot Mic PTT), J210.R, J212.PTT-2
- new net: J201.35 (Pilot Mic Lo), J210.S, J211.6, J212.PTT-1
- new net: J201.40 (Pass. Phone L), J213.R, J214.R
- new net: J201.41 (Pass. Phones R), J213.T, J214.T
- new net: J201.42 (Pass. Phone Lo), J213.S, J214.S
- new net: J209.6 (Copilot Trim Down Button), J227.DOWN
- new net: J209.13 (Copilot Trim Left Button), J227.LEFT
- new net: J205.34 (CoPilot Mic Lo), J223.6, J226.S, J227.PTT-2
- new net: J209.12 (Copilot Trim Right Button), J227.RIGHT
- new net: J209.5 (Copilot Trim Up Button), J227.UP
- new net: J209.14 (Roll Trim Motor Output 1), J234.1
- new net: J209.15 (Roll Trim Motor Output 2), J234.2
- new net: J206.6 (Serial 2 TX), J228.6, J229.6, J231.2
- new net: J206.5 (Serial 2 RX), J228.5, J229.5, J231.3
- new net: J216.23 (VOR/ILS Arinc Out B), J219.10
- new net: J216.24 (VOR/ILS Arinc Out A), J219.22
- new net: J209.10 (Pilot Trim Right Button), J212.RIGHT
- new net: J209.11 (Pilot Trim Left Button), J212.LEFT
- new net: J209.3 (Pilot Trim Up Button), J212.UP
- new net: J209.4 (Pilot Trim Down Button), J212.DOWN
- new net: J209.7 (Pitch Trim Motor Output 1), J233.1
- new net: J209.8 (Pitch Trim Motor Output 2), J233.2
- new net: J215.27 (Com Remote Transfer), J218.COM_1
- new net: J205.20 (COM Swap), J218.COM_SWAP
- new net: J206.3 (Serial 1 RX), J228.3, J229.3, J232.20
- new net: J206.4 (Serial 1 TX), J228.4, J229.4, J232.22
- new net: J205.3 (CoPlilot Phones L), J222.R, J223.3
- new net: J205.2 (CoPilot Phones Lo), J222.S, J223.2
- new net: J205.4 (CoPilot Phones R), J222.T, J223.4
- new net: J205.1 (Pilot Phones Lo), J211.2, J221.S
- new net: J205.15 (Alert 2 Audio Hi), J206.13, J206.31, J228.13, J228.31, J229.13, J229.31
- new net: J205.16 (Pilot Phones L), J211.3, J221.R
- new net: J205.31 (Pilot Phones R), J211.4, J221.T
- new net: J205.32 (Copilot Mic HI), J223.5, J226.T
- new net: J205.35 (Pass. Mic Hi), J224.T
- new net: J205.36 (Pass. Mic Lo), J224.S
- new net: J205.37 (Pass. 2 Mic Hi), J225.T
- new net: J205.38 (Pass. 2 Mic Lo), J225.S
- new net: J215.30 (POWER), J215.43, J215.44
- new net: J215.37 (GROUND), J215.38, J215.40
- new net: J228.1 (POWER), J228.20
- new net: J206.10 (GPS RS-232 In 4), J228.10 (Serial 4 TX), J229.10, J235.25
- new net: J228.21 (GROUND), J228.22
- new net: J206.9 (GPS RS-232 Out 4), J228.9, J229.9
- new net: J229.21 (GROUND), J229.22
- new net AG: J202.12 (GROUND IN), J206.21 (GROUND), J207.14 (GROUND), J208.5 (Ground), J209.2 (Ground -), J219.20 (Ground), J231.4 (Ground)
- new net ELT BUZZER: J204.8 (Buzzer Power Out)
Other:
- note added: "Wht/Brn"
- note added: "Wht/Grn"
- moved on the sheet: J206, J207, J208

Commit message: Record the owner's second round of answers; add OnSpeed and EMS sheets
24 recorded changes now, from the owner:

- OnSpeed is a Gen2v4 box on a DB-25 harness. Its pinout in sys-34 matches
  Phil's Gen2v4 aircraft harness drawing pin for pin, so the as-installed
  harness gets its own sheet: power from the essential bus through a 1 A
  blade fuse, SkyView Serial 4 TX in, right audio channel as mono into GMA
  245 Alert 3, flap position spliced into the VP-X flap sensor wire, and
  the button, LED and volume pot on a 6-conductor control cable.
- The CO detector is installed and powered. Only its audio and EMS data
  wires were cut - the audio input now carries OnSpeed and the EMS pin
  carries the MZ-30. sys-42 said it was not installed; corrected.
- EMS pin 31 is on the DB37 - the EMS's other connector has only 25 pins.
- COM 2 flip/flop has been wired to the grips since the build; the 2017
  drawing omits it. Recorded, with its return pin still to confirm.
- The GTN serial cut, OnSpeed, USB and MZ-30 work dates to about February
  2026.

Cross-sheet references follow the SteinAir convention: each sheet names
the far end as a label (ONSPEED DB25-10 on one side, GMA245 J1-29 on the
other).

sys-34 corrected: OnSpeed audio goes straight to the GMA 245, not through
the SkyView; power is from the essential bus on 1 A, not from the PFD on
2 A; the left audio channel is unused.

Five sheets, all verifying clean against their as-built wire lists.

Co-Authored-By: Claude Opus 5.5 <noreply@anthropic.com>
Claude-Session: https://claude.ai/code/session_015SpGdnvPFhutgEDurpngu2
Parts:
- removed J235: ONSPEED, symbol n720ak:ONSPEED
Connections:
- net ONSPEED DB25-25: now reaches J206.10 (Serial 4 TX), J228.10 (Serial 4 TX), J229.10
- new net ONSPEED DB25-10: J201.29 (Alert 3 Audio Hi)
Other:
- note added: "Gray"
- moved on the sheet: J202, J203, J204, J205, J206, J207, J208, J209, J210, J211, J212, J213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

Commit message: Record the third round of answers
- COM 2 flip/flop button returns to SV-COM-PANEL pin 3 (Ground out), on
  the owner's best recollection - recorded as unverified.
- OnSpeed's audio ground (pin 20) is tied to a ground pin in its own plug.
  GMA 245 Alert 3,4 Audio Lo (J1-43) is not connected, so the Alert 3
  input is single-ended.
- A panel switch disables the copilot grip trim by breaking the buttons'
  common. It is on neither SteinAir sheet, so it is recorded but flagged
  rather than drawn as a guess.
- AP disconnect is on both grips in parallel, as drawn.

Co-Authored-By: Claude Opus 5.5 <noreply@anthropic.com>
Claude-Session: https://claude.ai/code/session_015SpGdnvPFhutgEDurpngu2
Connections:
- new net: J218.COM_2_FLIP-FLOP, J230.7 (Ext flip/Flop)
- new net: J218.COM_2_FLIP-FLOP_RTN (Ground out), J230.3
Other:
- moved on the sheet: J210, J211, J212, J213, J214, J215, J216, J217, J219, J220, J221, J222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
