File: kicad/n720ak/SV.kicad_sch (KiCad schematic)
At the start: 34 parts, among them J201 GMA245 J1, J202 SV-COM C25 DB15, J203 GTN P1001, J204 ARTEX 345 ELT DB15, J205 GMA245 J2, J206 SV-HDX1100 (PFD2 – RIGHT #3) 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, J207 SV-XPNDR-261 DB-25M, J208 CO DETECTOR 452-101-011 DB9, J209 SV-AP-PANEL DB-15, J210 PILOT MIC JACK, J211 PILOT BOSE, J212 PILOT GRIP, J213 PASSENGER PHONE JACK 1, J214 PASSENGER PHONE JACK 2, J215 GTN 650 P1003, J216 GTN P1004, J217 MH OXYGEN CONTROL HEAD, J218 GRIPS, J219 Skyview ARINC DB25, J220 R-XPNDR-GPS (1.21 kOhm series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, J221 PILOT PHONE JACK, J222 COPILOT PHONE JACK, J223 COPILOT BOSE, J224 PASSENGER MIC JACK 1, J225 PASSENGER MIC JACK 2, J226 COPILOT MIC JACK, J227 COPILOT GRIP, J228 SV-HDX1100 (PFD - LEFT #1) DB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, J229 SV-HDX800 (MFD – CENTER #2) D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, J230 SV-COM-PANEL DB15, J231 SV-ADSB-472 DB9, J232 VP-X SPORT J1, J233 PITCH TRIM SERVO MOTOR, J234 ROLL TRIM SERVO MOTOR

Commit message: Build wing, terminal-block and EMS wire lists from the handbook tables
The wings, the under-seat terminal blocks and the EMS-220's 37-pin connector
are on no SteinAir drawing. Their only record is the owner's typed build
notes in sys-24 and sys-33. scripts/wirelist_handbook.py reads those tables
directly, so the WING and EMS wire lists cannot drift from the handbook.
Every join across connectors records what it rests on: matching bundle and
colour, a function named at both ends, or a manufacturer colour code (Dynon
servo pigtail, Ray Allen trim sensor leads). A join none of those settles
is flagged with the question that would settle it.

- KiCad: new WING sheet, full EMS sheet. The project netlist is now verified
  as a whole, which proves the cross-sheet labels merge (EMS pin 10 reaches
  the roll trim sensor through TB-L 3 and wing-root pin 12)
- INSPECT.md groups rows by question and picks up "Confirm at inspection"
  notes: 14 items
- SV trim motor outputs become labels that join TB-L on the WING sheet
- changes.tsv: CO detector RMA replacement (452-101-012, Dec 2025), its EFIS
  wire on EMS 31 and that wire's removal; C011 now names MZ-30 output Molex
  pin 5, 2026-03
- sys-33: AeroSun Vx colour table corrected to the Rev C manual (blue =
  taxi, yellow = wig-wag, green = sync), which matches TB-R 3's green pair
- sys-24: EMS pins 36/37 added to the unused table

Co-Authored-By: Claude Opus 5.5 <noreply@anthropic.com>
Claude-Session: https://claude.ai/code/session_015SpGdnvPFhutgEDurpngu2
Parts:
- removed J201: GMA245 J1, symbol n720ak:GMA245_J1
- removed J202: SV-COM C25 DB15, symbol n720ak:SV-COM_C25_DB15
- removed J203: GTN P1001, symbol n720ak:GTN_P1001
- removed J204: ARTEX 345 ELT DB15, symbol n720ak:ARTEX_345_ELT_DB15
- removed J205: GMA245 J2, symbol n720ak:GMA245_J2
- removed J206: SV-HDX1100 (PFD2 – RIGHT #3) DB37, symbol n720ak:SV-HDX1100__PFD2___RIGHT__3__DB37
- removed J207: SV-XPNDR-261 DB-25M, symbol n720ak:SV-XPNDR-261_DB-25M
- removed J208: CO DETECTOR 452-101-011 DB9, symbol n720ak:CO_DETECTOR_452-101-011_DB9
- removed J209: SV-AP-PANEL DB-15, symbol n720ak:SV-AP-PANEL_DB-15
- removed J210: PILOT MIC JACK, symbol n720ak:PILOT_MIC_JACK
- removed J211: PILOT BOSE, symbol n720ak:PILOT_BOSE
- removed J212: PILOT GRIP, symbol n720ak:PILOT_GRIP
- removed J213: PASSENGER PHONE JACK 1, symbol n720ak:PASSENGER_PHONE_JACK_1
- removed J214: PASSENGER PHONE JACK 2, symbol n720ak:PASSENGER_PHONE_JACK_2
- removed J215: GTN 650 P1003, symbol n720ak:GTN_650_P1003
- removed J216: GTN P1004, symbol n720ak:GTN_P1004
- removed J217: MH OXYGEN CONTROL HEAD, symbol n720ak:MH_OXYGEN_CONTROL_HEAD
- removed J218: GRIPS, symbol n720ak:GRIPS
- removed J219: Skyview ARINC DB25, symbol n720ak:Skyview_ARINC_DB25
- removed J220: R-XPNDR-GPS (1.21 kOhm series resistor), symbol n720ak:R-XPNDR-GPS__1.21_kOhm_series_resistor_
- removed J221: PILOT PHONE JACK, symbol n720ak:PILOT_PHONE_JACK
- removed J222: COPILOT PHONE JACK, symbol n720ak:COPILOT_PHONE_JACK
- removed J223: COPILOT BOSE, symbol n720ak:COPILOT_BOSE
- removed J224: PASSENGER MIC JACK 1, symbol n720ak:PASSENGER_MIC_JACK_1
- removed J225: PASSENGER MIC JACK 2, symbol n720ak:PASSENGER_MIC_JACK_2
- removed J226: COPILOT MIC JACK, symbol n720ak:COPILOT_MIC_JACK
- removed J227: COPILOT GRIP, symbol n720ak:COPILOT_GRIP
- removed J228: SV-HDX1100 (PFD - LEFT #1) DB37, symbol n720ak:SV-HDX1100__PFD_-_LEFT__1__DB37
- removed J229: SV-HDX800 (MFD – CENTER #2) DB37, symbol n720ak:SV-HDX800__MFD___CENTER__2__DB37
- removed J230: SV-COM-PANEL DB15, symbol n720ak:SV-COM-PANEL_DB15
- removed J231: SV-ADSB-472 DB9, symbol n720ak:SV-ADSB-472_DB9
- removed J232: VP-X SPORT J1, symbol n720ak:VP-X_SPORT_J1
- removed J233: PITCH TRIM SERVO MOTOR, symbol n720ak:PITCH_TRIM_SERVO_MOTOR
- removed J234: ROLL TRIM SERVO MOTOR, symbol n720ak:ROLL_TRIM_SERVO_MOTOR
- added J201: PILOT MIC JACK, symbol n720ak:PILOT_MIC_JACK
- added J202: PILOT BOSE, symbol n720ak:PILOT_BOSE
- added J203: PILOT GRIP, symbol n720ak:PILOT_GRIP
- added J204: PASSENGER PHONE JACK 1, symbol n720ak:PASSENGER_PHONE_JACK_1
- added J205: PASSENGER PHONE JACK 2, symbol n720ak:PASSENGER_PHONE_JACK_2
- added J206: GTN 650 P1003, symbol n720ak:GTN_650_P1003
- added J207: GTN P1004, symbol n720ak:GTN_P1004
- added J208: MH OXYGEN CONTROL HEAD, symbol n720ak:MH_OXYGEN_CONTROL_HEAD
- added J209: GRIPS, symbol n720ak:GRIPS
- added J210: Skyview ARINC DB25, symbol n720ak:Skyview_ARINC_DB25
- added J211: R-XPNDR-GPS (1.21 kOhm series resistor), symbol n720ak:R-XPNDR-GPS__1.21_kOhm_series_resistor_
- added J212: PILOT PHONE JACK, symbol n720ak:PILOT_PHONE_JACK
- added J213: COPILOT PHONE JACK, symbol n720ak:COPILOT_PHONE_JACK
- added J214: COPILOT BOSE, symbol n720ak:COPILOT_BOSE
- added J215: PASSENGER MIC JACK 1, symbol n720ak:PASSENGER_MIC_JACK_1
- added J216: PASSENGER MIC JACK 2, symbol n720ak:PASSENGER_MIC_JACK_2
- added J217: COPILOT MIC JACK, symbol n720ak:COPILOT_MIC_JACK
- added J218: COPILOT GRIP, symbol n720ak:COPILOT_GRIP
- added J219: SV-HDX1100 (PFD - LEFT #1) DB37, symbol n720ak:SV-HDX1100__PFD_-_LEFT__1__DB37
- added J220: SV-HDX800 (MFD – CENTER #2) DB37, symbol n720ak:SV-HDX800__MFD___CENTER__2__DB37
- added J221: SV-COM-PANEL DB15, symbol n720ak:SV-COM-PANEL_DB15
- added J222: SV-ADSB-472 DB9, symbol n720ak:SV-ADSB-472_DB9
- added J223: VP-X SPORT J1, symbol n720ak:VP-X_SPORT_J1
- added J224: GMA245 J1, symbol n720ak:GMA245_J1
- added J225: SV-COM C25 DB15, symbol n720ak:SV-COM_C25_DB15
- added J226: GTN P1001, symbol n720ak:GTN_P1001
- added J227: ARTEX 345 ELT DB15, symbol n720ak:ARTEX_345_ELT_DB15
- added J228: GMA245 J2, symbol n720ak:GMA245_J2
- added J229: SV-HDX1100 (PFD2 – RIGHT #3) DB37, symbol n720ak:SV-HDX1100__PFD2___RIGHT__3__DB37
- added J230: SV-XPNDR-261 DB-25M, symbol n720ak:SV-XPNDR-261_DB-25M
- added J231: CO DETECTOR 452-101-012 DB9, symbol n720ak:CO_DETECTOR_452-101-012_DB9
- added J232: SV-AP-PANEL DB-15, symbol n720ak:SV-AP-PANEL_DB-15
Connections:
- net 7 8: now also J227.14 (External On), J227.3 (2-Wire Remote Switch)
- net AG: now also J210.20 (Ground), J222.4 (Ground), J225.12 (GROUND IN), J229.21 (GROUND), J230.14 (GROUND), J231.5 (Ground), J232.2 (Ground -)
- net ELT BUZZER: now also J227.8 (Buzzer Power Out)
- net GROUND: now also J227.7 (Ground), J229.22 (GROUND)
- net GTN CONFIG MODULE: now also J226.62 (Config Mod Data), J226.63 (Config Mod Clock), J226.64 (Config Mod Ground), J226.65 (Config Mod Power)
- net GTN FAN: now also J226.43 (Fan Ground), J226.58 (Fan Tach In), J226.59 (Fan Power)
- net ONSPEED DB25-10: now also J224.29 (Alert 3 Audio Hi)
- net ONSPEED DB25-25: now also J219.10 (Serial 4 TX), J220.10, J229.10 (Serial 4 TX)
- net SV-GPS-250: now also J219.11, J219.12, J219.24, J219.29, J220.11, J220.12, J220.24, J220.29, J229.11 (Serial 5 RX), J229.12 (Serial 5 TX), J229.24 (SV-GPS-250 Ground), J229.29 (SV-GPS-250 Power)
- net USB Socket: now also J219.16 (USB Power), J219.17 (USB Ground (withshield)), J219.18 (USB Data -), J219.19 (USB Data +), J220.16 (USB Power), J220.17 (USB Ground (withshield)), J220.18 (USB Data -), J220.19 (USB Data +), J229.16 (USB Power), J229.17 (USB Ground (withshield)), J229.18 (USB Data -), J229.19 (USB Data +)
- net VP-X J10-2: now also J229.1 (POWER), J229.20
- net VP-X J10-4: now also J202.1, J214.1, J228.8 (11-33 VDC), J228.9
- net VP-X J10-7: now also J222.1 (Power), J230.15 (POWER)
- net VP-X J10-8: now also J231.1 (Power)
- net VP-X J12-10: now also J232.9 (Power In +)
- net VP-X J12-7: now also J225.8 (POWER IN)
- net VP-X J12-9: now also J220.1 (POWER), J220.20
- new net: J213.S, J214.2, J228.2 (CoPilot Phones Lo)
- new net: J213.R, J214.3, J228.3 (CoPlilot Phones L)
- new net: J213.T, J214.4, J228.4 (CoPilot Phones R)
- new net: J214.5, J217.T, J228.32 (Copilot Mic HI)
- new net: J214.6, J217.S, J218.PTT-2, J228.34 (CoPilot Mic Lo)
- new net: J202.2, J212.S, J228.1 (Pilot Phones Lo)
- new net: J202.3, J212.R, J228.16 (Pilot Phones L)
- new net: J202.4, J212.T, J228.31 (Pilot Phones R)
- new net: J201.T, J202.5, J224.33 (Pilot Mic Hi)
- new net: J201.S, J202.6, J203.PTT-1, J224.35 (Pilot Mic Lo)
- new net: J221.1, J225.7 (SV-COM POWER)
- new net: J221.2, J225.13 (SV COM GROUND)
- new net: J209.COM_2_FLIP-FLOP_RTN (Ground out), J221.3
- new net: J221.4, J225.6 (SV-COM-PANEL DATA IN)
- new net: J221.5, J225.14 (SV COM DATA OUT)
- new net: J221.6, J225.3 (SV COM PANEL ENABLE)
- new net: J209.COM_2_FLIP-FLOP, J221.7 (Ext flip/Flop)
- new net: J219.1 (POWER), J219.20
- new net: J219.13, J219.31, J220.13, J220.31, J228.15 (Alert 2 Audio Hi), J229.13, J229.31
- new net: J219.21 (GROUND), J219.22
- new net: J219.3, J220.3, J223.20, J229.3 (Serial 1 RX)
- new net: J219.30, J220.30, J228.14 (Alert 2 Audio Lo), J229.30
- new net: J219.4, J220.4, J223.22, J229.4 (Serial 1 TX)
- new net: J219.5, J220.5, J222.3, J229.5 (Serial 2 RX)
- new net: J219.6, J220.6, J222.2, J229.6 (Serial 2 TX)
- new net: J219.7, J220.7, J229.7, J230.7 (Serial Out)
- new net: J219.8, J220.8, J229.8, J230.5 (Serial In)
- new net: J219.9, J220.9, J229.9 (Serial 4 RX)
- new net: J218.DOWN, J232.6 (Copilot Trim Down Button)
- new net: J218.LEFT, J232.13 (Copilot Trim Left Button)
- new net: J217.R, J218.PTT-1, J228.33 (CoPilot Mic PTT)
- new net: J218.RIGHT, J232.12 (Copilot Trim Right Button)
- new net: J218.UP, J232.5 (Copilot Trim Up Button)
- new net: J206.18, J206.20, J224.10 (Com 1 Lo)
- new net: J206.5, J224.11 (Com 1 Mic HI)
- new net: J206.11, J224.12 (Com 1 Mic Key)
- new net: J224.13, J225.10 (PHONES OUT)
- new net: J224.14, J225.2 (MIC LO), J225.9
- new net: J224.15, J225.1 (MIC HI)
- new net: J207.16, J224.17 (Nav 1 Audio Hi)
- new net: J207.17, J224.18 (Nav 1 Lo)
- new net: J224.30, J225.5 (PTT IN)
- new net: J224.31 (Alert 1 Audio Hi), J226.4
- new net: J224.32 (Alert 1 Audio Lo), J226.23
- new net: J201.R, J203.PTT-2, J224.34 (Pilot Mic PTT)
- new net: J204.R, J205.R, J224.40 (Pass. Phone L)
- new net: J204.T, J205.T, J224.41 (Pass. Phones R)
- new net: J204.S, J205.S, J224.42 (Pass. Phone Lo)
- new net: J208.DB25-9, J224.44 (Alert 4 Audio Hi)
- new net: J206.7, J224.9 (Com 1 Audio Hi)
- new net: J203.RIGHT, J232.10 (Pilot Trim Right Button)
- new net: J203.LEFT, J232.11 (Pilot Trim Left Button)
- new net: J203.UP, J232.3 (Pilot Trim Up Button)
- new net: J203.DOWN, J232.4 (Pilot Trim Down Button)
- new net: J210.23, J226.10 (GPS ARINC 429 OUT 1A)
- new net: J207.51, J207.52, J226.19 (POWER 1), J226.20
- new net: J210.11, J226.29 (GPS ARINC 429 OUT 1B)
- new net: J210.24, J226.48 (GPS ARINC 429 IN 1A)
- new net: J226.6 (GPS RS-232 Out 3), J227.9
- new net: J210.12, J226.67 (GPS ARINC 429 IN 1B)
- new net: J211.1, J226.7 (GPS RS-232 Out 2)
- new net: J207.61, J207.62, J226.77 (GROUND), J226.78
- new net: J210.3, J226.8 (GPS RS-232 Out 1)
- new net: J227.12, J227.5 (G-Switch Loop)
- new net: J206.27 (Com Remote Transfer), J209.COM_1
- new net: J206.30 (POWER), J206.43, J206.44
- new net: J206.37 (GROUND), J206.38, J206.40
- new net: J230.1 (Jumper), J230.2
- new net: J230.12 (Jumper), J230.13
- new net: J211.2, J230.3 (GPS In (ADS-B))
- new net: J207.23 (VOR/ILS Arinc Out B), J210.10
- new net: J207.24 (VOR/ILS Arinc Out A), J210.22
- new net: J228.10 (Ground), J228.11
- new net: J209.COM_SWAP, J228.20 (COM Swap)
- new net: J215.T, J228.35 (Pass. Mic Hi)
- new net: J215.S, J228.36 (Pass. Mic Lo)
- new net: J216.T, J228.37 (Pass. 2 Mic Hi)
- new net: J216.S, J228.38 (Pass. 2 Mic Lo)
- new net: J220.21 (GROUND), J220.22
- new net PITCH TRIM MOTOR A: J232.7 (Pitch Trim Motor Output 1)
- new net PITCH TRIM MOTOR B: J232.8 (Pitch Trim Motor Output 2)
- new net ROLL TRIM MOTOR A: J232.14 (Roll Trim Motor Output 1)
- new net ROLL TRIM MOTOR B: J232.15 (Roll Trim Motor Output 2)
